Commit message: Corregido errores en el gazebo

File: kuka_kr5_arc/kr5_gazebo/urdf/gazebo.xacro (robot description, xacro)
@@ -3,5 +3,5 @@
   <!-- KR5 -->
   <xacro:include filename="$(find kr5_gazebo)/urdf/gazebo_transmission.xacro"/>
-  <xacro:kuka_kr5_robot prefix=""/>
+  <xacro:kuka_kr5 prefix=""/>
   <!-- Fix robot to Gazebo world -->
   <link name="world"/>

File: kuka_kr5_arc/kr5_gazebo/urdf/gazebo_transmission.xacro (robot description, xacro)
@@ -2,111 +2,111 @@
 <robot xmlns:xacro="http://wiki.ros.org/xacro">
     <xacro:include filename="$(find kr5_description/urdf/kr5_arc_macro.xacro)"/>
-    <xacro:macro name="kuka_kr5_robot" params="prefix"/>
-    <!-- get URDF description of KUKA KR5 model -->
-    <xacro:kuka_kr5_robot prefix="${prefix}" />
-    <!-- transmission list -->
-    <transmission name="${prefix}tran1">
-        <robotNamespace>/${prefix}</robotNamespace>
-        <type>transmission_interface/SimpleTransmission</type>
-        <joint name="${prefix}joint_a1">
-            <hardwareInterface>hardware_interface/PositionJointInterface</hardwareInterface>
-        </joint>
-        <actuator name="${prefix}motor1">
-            <mechanicalReduction>1</mechanicalReduction>
-            <hardwareInterface>hardware_interface/PositionJointInterface</hardwareInterface>
-        </actuator>
-    </transmission>
-    <transmission name="${prefix}tran2">
-        <robotNamespace>/${prefix}</robotNamespace>
-        <type>transmission_interface/SimpleTransmission</type>
-        <joint name="${prefix}joint_a2">
-            <hardwareInterface>hardware_interface/PositionJointInterface</hardwareInterface>
-        </joint>
-        <actuator name="${prefix}motor2">
-            <mechanicalReduction>1</mechanicalReduction>
-            <hardwareInterface>hardware_interface/PositionJointInterface</hardwareInterface>
-        </actuator>
-    </transmission>
-    <transmission name="${prefix}tran3">
-        <robotNamespace>/${prefix}</robotNamespace>
-        <type>transmission_interface/SimpleTransmission</type>
-        <joint name="${prefix}joint_a3">
-            <hardwareInterface>hardware_interface/PositionJointInterface</hardwareInterface>
-        </joint>
-        <actuator name="${prefix}motor3">
-            <mechanicalReduction>1</mechanicalReduction>
-            <hardwareInterface>hardware_interface/PositionJointInterface</hardwareInterface>
-        </actuator>
-    </transmission>
-    <transmission name="${prefix}tran4">
-        <robotNamespace>/${prefix}</robotNamespace>
-        <type>transmission_interface/SimpleTransmission</type>
-        <joint name="${prefix}joint_a4">
-            <hardwareInterface>hardware_interface/PositionJointInterface</hardwareInterface>
-        </joint>
-        <actuator name="${prefix}motor4">
-            <mechanicalReduction>1</mechanicalReduction>
-            <hardwareInterface>hardware_interface/PositionJointInterface</hardwareInterface>
-        </actuator>
-    </transmission>
-    <transmission name="${prefix}tran5">
-        <robotNamespace>/${prefix}</robotNamespace>
-        <type>transmission_interface/SimpleTransmission</type>
-        <joint name="${prefix}joint_a5">
-            <hardwareInterface>hardware_interface/PositionJointInterface</hardwareInterface>
-        </joint>
-        <actuator name="${prefix}motor5">
-            <mechanicalReduction>1</mechanicalReduction>
-            <hardwareInterface>hardware_interface/PositionJointInterface</hardwareInterface>
-        </actuator>
-    </transmission>
-    <transmission name="${prefix}tran6">
-        <robotNamespace>/${prefix}</robotNamespace>
-        <type>transmission_interface/SimpleTransmission</type>
-        <joint name="${prefix}joint_a6">
-            <hardwareInterface>hardware_interface/PositionJointInterface</hardwareInterface>
-        </joint>
-        <actuator name="${prefix}motor6">
-            <mechanicalReduction>1</mechanicalReduction>
-            <hardwareInterface>hardware_interface/PositionJointInterface</hardwareInterface>
-        </actuator>
-    </transmission>
-    <!-- end of transmission list -->
-    <!-- Gazebo-specific link properties -->
-    <gazebo reference="${prefix}base_link">
-        <material>Gazebo/Black</material>
-        <turnGravityOff>true</turnGravityOff>
-    </gazebo>
-    <gazebo reference="${prefix}link_1">
-        <material>Gazebo/Orange</material>
-        <turnGravityOff>true</turnGravityOff>
-    </gazebo>
-    <gazebo reference="${prefix}link_2">
-        <material>Gazebo/Orange</material>
-        <turnGravityOff>true</turnGravityOff>
-    </gazebo>
-    <gazebo reference="${prefix}link_3">
-        <material>Gazebo/Orange</material>
-        <turnGravityOff>true</turnGravityOff>
-    </gazebo>
-    <gazebo reference="${prefix}link_4">
-        <material>Gazebo/Orange</material>
-        <turnGravityOff>true</turnGravityOff>
-    </gazebo>
-    <gazebo reference="${prefix}link_5">
-        <material>Gazebo/Grey</material>
-        <turnGravityOff>true</turnGravityOff>
-    </gazebo>
-    <gazebo reference="${prefix}link_6">
-        <material>Gazebo/Grey</material>
-        <turnGravityOff>true</turnGravityOff>
-    </gazebo>
-    <!-- ros_control plugin -->
-    <gazebo>
-        <plugin name="gazebo_ros_control" filename="libgazebo_ros_control.so">
+    <xacro:macro name="kuka_kr5_robot" params="prefix">
+        <!-- get URDF description of KUKA KR5 model -->
+        <xacro:kuka_kr5 prefix="${prefix}" />
+        <!-- transmission list -->
+        <transmission name="${prefix}tran1">
             <robotNamespace>/${prefix}</robotNamespace>
-            <robotSimType>gazebo_ros_control/DefaultRobotHWSim</robotSimType>
-        </plugin>
-    </gazebo>
-</xacro:macro>
+            <type>transmission_interface/SimpleTransmission</type>
+            <joint name="${prefix}joint_a1">
+                <hardwareInterface>hardware_interface/PositionJointInterface</hardwareInterface>
+            </joint>
+            <actuator name="${prefix}motor1">
+                <mechanicalReduction>1</mechanicalReduction>
+                <hardwareInterface>hardware_interface/PositionJointInterface</hardwareInterface>
+            </actuator>
+        </transmission>
+        <transmission name="${prefix}tran2">
+            <robotNamespace>/${prefix}</robotNamespace>
+            <type>transmission_interface/SimpleTransmission</type>
+            <joint name="${prefix}joint_a2">
+                <hardwareInterface>hardware_interface/PositionJointInterface</hardwareInterface>
+            </joint>
+            <actuator name="${prefix}motor2">
+                <mechanicalReduction>1</mechanicalReduction>
+                <hardwareInterface>hardware_interface/PositionJointInterface</hardwareInterface>
+            </actuator>
+        </transmission>
+        <transmission name="${prefix}tran3">
+            <robotNamespace>/${prefix}</robotNamespace>
+            <type>transmission_interface/SimpleTransmission</type>
+            <joint name="${prefix}joint_a3">
+                <hardwareInterface>hardware_interface/PositionJointInterface</hardwareInterface>
+            </joint>
+            <actuator name="${prefix}motor3">
+                <mechanicalReduction>1</mechanicalReduction>
+                <hardwareInterface>hardware_interface/PositionJointInterface</hardwareInterface>
+            </actuator>
+        </transmission>
+        <transmission name="${prefix}tran4">
+            <robotNamespace>/${prefix}</robotNamespace>
+            <type>transmission_interface/SimpleTransmission</type>
+            <joint name="${prefix}joint_a4">
+                <hardwareInterface>hardware_interface/PositionJointInterface</hardwareInterface>
+            </joint>
+            <actuator name="${prefix}motor4">
+                <mechanicalReduction>1</mechanicalReduction>
+                <hardwareInterface>hardware_interface/PositionJointInterface</hardwareInterface>
+            </actuator>
+        </transmission>
+        <transmission name="${prefix}tran5">
+            <robotNamespace>/${prefix}</robotNamespace>
+            <type>transmission_interface/SimpleTransmission</type>
+            <joint name="${prefix}joint_a5">
+                <hardwareInterface>hardware_interface/PositionJointInterface</hardwareInterface>
+            </joint>
+            <actuator name="${prefix}motor5">
+                <mechanicalReduction>1</mechanicalReduction>
+                <hardwareInterface>hardware_interface/PositionJointInterface</hardwareInterface>
+            </actuator>
+        </transmission>
+        <transmission name="${prefix}tran6">
+            <robotNamespace>/${prefix}</robotNamespace>
+            <type>transmission_interface/SimpleTransmission</type>
+            <joint name="${prefix}joint_a6">
+                <hardwareInterface>hardware_interface/PositionJointInterface</hardwareInterface>
+            </joint>
+            <actuator name="${prefix}motor6">
+                <mechanicalReduction>1</mechanicalReduction>
+                <hardwareInterface>hardware_interface/PositionJointInterface</hardwareInterface>
+            </actuator>
+        </transmission>
+        <!-- end of transmission list -->
+        <!-- Gazebo-specific link properties -->
+        <gazebo reference="${prefix}base_link">
+            <material>Gazebo/Black</material>
+            <turnGravityOff>true</turnGravityOff>
+        </gazebo>
+        <gazebo reference="${prefix}link_1">
+            <material>Gazebo/Orange</material>
+            <turnGravityOff>true</turnGravityOff>
+        </gazebo>
+        <gazebo reference="${prefix}link_2">
+            <material>Gazebo/Orange</material>
+            <turnGravityOff>true</turnGravityOff>
+        </gazebo>
+        <gazebo reference="${prefix}link_3">
+            <material>Gazebo/Orange</material>
+            <turnGravityOff>true</turnGravityOff>
+        </gazebo>
+        <gazebo reference="${prefix}link_4">
+            <material>Gazebo/Orange</material>
+            <turnGravityOff>true</turnGravityOff>
+        </gazebo>
+        <gazebo reference="${prefix}link_5">
+            <material>Gazebo/Grey</material>
+            <turnGravityOff>true</turnGravityOff>
+        </gazebo>
+        <gazebo reference="${prefix}link_6">
+            <material>Gazebo/Grey</material>
+            <turnGravityOff>true</turnGravityOff>
+        </gazebo>
+        <!-- ros_control plugin -->
+        <gazebo>
+            <plugin name="gazebo_ros_control" filename="libgazebo_ros_control.so">
+                <robotNamespace>/${prefix}</robotNamespace>
+                <robotSimType>gazebo_ros_control/DefaultRobotHWSim</robotSimType>
+            </plugin>
+        </gazebo>
+    </xacro:macro>
 </robot>
